File: acl-adapter.brd (EAGLE design)
At the start: 79 parts, among them IC1 UCC27712, IC2 UCC28780, IC3 TL431, Q1 TK8Q60, Q2 TK8Q60, Q3 2N7002, Q5 TLP621-1, T1 COMMON_FILTER-SU10VFC, T2 TRANSFORMAER_FLYBACK-PQ2620-A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

Commit message: ボード図だいたい
Parts:
- added C22: 100p, my_rcl:1608
- added HT1, HT2, HT3: HEATSINK-2, my_connector:HEATSINK2
- added R27: 10, my_rcl:1608
- C4, C6: device my_rcl:2012 -> my_rcl:1608
- D5: device my_rcl:D0207/2V -> my_rcl:D0204/7
- moved C4 159.3 mm to (53.0, 4.76), flipped to the bottom, turned to 90 degrees
- moved D3 155.2 mm to (61.3, 18.1), flipped to the bottom
- moved D4 153.9 mm to (62.9, 14.4), flipped to the bottom, turned to 270 degrees
- moved C6 149.9 mm to (49.2, 10.5), flipped to the bottom, turned to 270 degrees
- moved R14 143.1 mm to (60.6, 21.0), flipped to the bottom, turned to 90 degrees
- moved R16 137.1 mm to (57.1, 20.0), flipped to the bottom, turned to 180 degrees
- moved C5 134.0 mm to (48.9, 18.7), flipped to the bottom
- moved C12 115.9 mm to (58.7, 4.76), flipped to the bottom, turned to 90 degrees
- moved D1 61.1 mm to (40.0, 14.0), turned to 90 degrees
- moved T1 52.8 mm to (30.5, 16.2), turned to 90 degrees
- moved C1 37.0 mm to (31.8, 29.2), turned to 0 degrees
- moved R6 30.2 mm to (68.4, 9.68), turned to 90 degrees
- moved TP2 26.9 mm to (29.2, 39.4)
- moved C2 23.6 mm to (47.6, 31.8), turned to 180 degrees
- moved R5 23.2 mm to (62.5, 4.76), turned to 270 degrees
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Connections:
- new net N$30: C22.2, IC2.3, R27.1
- net FB: no longer D3.1
- net GND: now also HT1.HT1, HT3.HT1
- net N$1: now also TP2.1; no longer TP1.1
- net N$15: now also R27.2; no longer IC1.4, IC2.3
- net N$17: now also R19.1; no longer C15.2
- net N$2: now also F1.2; no longer TP2.1
- net N$3: now also TP1.1; no longer F1.2
- net N$6: now also C15.2; no longer R19.2
- net N$8: now also R19.2; no longer R19.1
- net PGND: now also C22.1, D3.1, HT2.HT1, IC1.4
Routing:
- net N$40: track 27.1 -> 65.1 mm
- net N$2: track 0.00 -> 34.3 mm
- net VDD: track 0.00 -> 34.0 mm, vias 0 -> 3
- net VP: track 18.8 -> 51.1 mm
- net REF: track 0.00 -> 28.6 mm
- net N$23: track 0.00 -> 25.9 mm
- net N$30: track 0.00 -> 23.7 mm
- net N$6: track 0.00 -> 22.8 mm
- net FB: track 0.00 -> 19.1 mm
- net N$17: track 0.00 -> 18.7 mm
- net PGND: track 0.00 -> 18.0 mm
- net RUN: track 0.00 -> 17.0 mm, vias 0 -> 2
- net N$3: track 0.00 -> 15.9 mm
- net SWS: track 0.00 -> 12.9 mm
- net HVG: track 0.00 -> 12.1 mm
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
Commit message: 基板ほぼできた
Parts:
- D2: device my_rcl:D0207/2V -> my_rcl:D0204/7
- moved TP1 26.1 mm to (3.17, 36.2)
- moved DR3 21.0 mm to (3.17, 3.17)
- moved F1 21.0 mm to (15.9, 38.7)
- moved C1 21.0 mm to (10.8, 29.8)
- moved SJ2 21.0 mm to (89.5, 6.35)
- moved T1 21.0 mm to (9.53, 16.5)
- moved R10 20.6 mm to (38.7, 35.9)
- moved D2 20.5 mm to (34.3, 24.8)
- moved SJ1 20.5 mm to (86.2, 6.35)
- moved C7 20.5 mm to (34.1, 26.0)
- moved C17 20.3 mm to (78.7, 19.7)
- moved C18 20.3 mm to (78.7, 30.5)
- moved C19 20.3 mm to (67.9, 4.76)
- moved D5 20.3 mm to (49.8, 9.53)
- moved D6 20.3 mm to (77.5, 8.89)
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Routing:
- net PGND: track 18.0 -> 61.8 mm
- net N$9: track 9.69 -> 30.9 mm
- net N$6: track 22.8 -> 30.9 mm
- net V+: track 8.64 -> 13.7 mm
- net N$10: track 8.18 -> 3.99 mm, vias 1 -> 0
- net N$17: track 18.7 -> 22.0 mm
- net N$23: track 25.9 -> 29.0 mm
- net N$18: track 6.69 -> 8.94 mm
- net N$3: track 15.9 -> 13.7 mm
- net N$8: track 0.00 -> 2.09 mm
- net N$40: track 65.1 -> 63.3 mm
- net N$22: track 0.00 -> 1.80 mm
- net N$2: track 34.3 -> 36.0 mm
- net N$30: track 23.7 -> 22.7 mm
- net N$4: track 5.26 -> 6.03 mm
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- added copper zone on layer 1, net GND
- added copper zone on layer 16, net GND
- added copper zone on layer 16, net N$17
- added copper zone on layer 16, net N$18
- added copper zone on layer 1, net N$23
- added copper zone on layer 16, net N$23
- added copper zone on layer 1, net N$6
- added copper zone on layer 16, net N$6
- added copper zone on layer 1, net PGND
- added copper zone on layer 16, net PGND
- added copper zone on layer 16, net V+
- added copper zone on layer 16, net V-
Other:
- board outline added: 98.4 x 49.5 mm

Commit message: できた
Parts:
- added C23: 1000p, my_rcl:1608
- added R28: 10, my_rcl:1608
- added R29: 1.5k, my_rcl:1608
- C10: value 22p -> 27p
- C7: value 0.1u -> 1u; device my_rcl:2012 -> my_rcl:1608
- R21, R22: value 1.5k -> 10k
- moved R12 4.92 mm to (27.1, 41.8)
- moved Q1 2.62 mm to (42.5, 40.0)
- moved R11 2.46 mm to (41.1, 41.9)
- moved R8 2.46 mm to (39.7, 37.3)
- moved HT2 1.93 mm to (28.6, 43.5)
- moved Q2 1.91 mm to (28.6, 40.0)
- moved DR3 0.90 mm to (3.81, 3.81)
- moved SJ2 0.57 mm to (89.9, 6.83)
- moved SJ1 0.50 mm to (86.4, 6.83)
- moved HT3 0.48 mm to (74.3, 43.5)
- moved HT1 0.16 mm to (77.5, 6.03)
- moved R22 0.16 mm to (61.9, 8.89)
- turned R9 to 180 degrees
Connections:
- new net N$31: D2.2, R28.1
- new net N$33: C23.1, R29.2
- net N$10: now also R28.2; no longer D2.2
- net N$29: now also R29.1
- net N$9: now also C23.2
Routing:
- net N$9: track 30.9 -> 35.3 mm
- net N$15: track 10.2 -> 13.2 mm
- net N$11: track 17.6 -> 15.0 mm
- net N$7: track 7.07 -> 4.53 mm
- net N$31: track 0.00 -> 2.17 mm
- net N$33: track 0.00 -> 1.85 mm
- net N$29: track 7.63 -> 9.38 mm
- net N$13: track 9.57 -> 7.88 mm
- net N$40: track 63.3 -> 61.9 mm
- net N$10: track 3.99 -> 4.69 mm
- net N$6: track 30.9 -> 30.4 mm
- net V+: track 13.7 -> 13.2 mm
- net PGND: track 61.8 -> 61.5 mm, vias 0 -> 39
Other:
- board text added: "ACF Power Supply"
- board text added: "ver 1"
