File: acf-adapter.brd (EAGLE design)
At the start: 98.4 x 49.5 mm, 87 parts, among them IC1 UCC27712, IC2 UCC28780, IC3 TL431, Q1 TK8Q60, Q2 TK8Q60, Q3 2N7002, Q5 TLP621-1, T1 COMMON_FILTER-SU10VFC, T2 TRANSFORMAER_FLYBACK-PQ2620-A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

Commit message: できた
Parts:
- Q1: value TK8Q60 -> 2SK3115
- Q2: value TK8Q60 -> TK13A60
- Q4: value (none) -> BSS127
- moved TP2 1.80 mm to (8.26, 41.3)
- moved F1 0.90 mm to (15.2, 38.1), turned to 0 degrees
- moved HT2 0.48 mm to (28.6, 44.0)
- moved HT1 0.32 mm to (77.5, 5.71)
- moved HT3 0.32 mm to (74.3, 43.8)
Routing:
- net N$2: track 36.0 -> 37.4 mm
- net N$1: track 6.89 -> 5.80 mm

Commit message: 微修正
Parts:
- R16: value 100 -> 120
- R2: value 250k -> 125k
