File: acf-adapter.brd (EAGLE design)
At the start: 98.4 x 49.5 mm, 87 parts, among them IC1 UCC27712, IC2 UCC28780, IC3 TL431, Q1 2SK3115, Q2 TK13A60, Q3 2N7002, Q4 BSS127, Q5 TLP621-1, T1 COMMON_FILTER-SU10VFC, T2 TRANSFORMAER_FLYBACK-PQ2620-A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

Commit message: 発注
Parts:
- added R30: 240k, my_rcl:1608
- R1: value 250k -> 240k
- R14: value 1M -> 240k
- R15: value 470k -> 240k
- R2: value 125k -> 120k
- R27: value 10 -> 120
- R8, R9: device my_rcl:1608 -> my_rcl:2012
- moved Q3 0.32 mm to (48.9, 5.71)
- moved R17 0.32 mm to (51.6, 5.71)
Connections:
- new net N$37: R15.1, R30.1
- net N$34: now also R30.2; no longer R15.1
Routing:
- net N$37: track 0.00 -> 1.91 mm
- net FB: track 19.1 -> 20.6 mm
- net N$34: track 4.45 -> 3.60 mm

Commit message: 微修正
Parts:
- C11: value 10u -> 47u
- C6: value 1u -> 0.1u
- C8: value 0.47u -> 0.1u
- R2: value 120k -> 47k
- R21: value 10k -> 1.5k
- R23: value 10k -> 47k
- R7: value 250k -> 240k
Changed lines of the file:
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@@
 <attribute name="VALUE" x="50.495" y="14.71" size="0.8128" layer="28" rot="MR0"/>
 </element>
-<element name="C11" library="my_rcl" package="2012" value="10u" x="42.545" y="10.4775" smashed="yes" rot="MR90">
+<element name="C11" library="my_rcl" package="2012" value="47u" x="42.545" y="10.4775" smashed="yes" rot="MR90">
 <attribute name="NAME" x="40.545" y="9.0775" size="0.8128" layer="26" rot="MR90"/>
 <attribute name="VALUE" x="43.945" y="9.0775" size="0.8128" layer="28" rot="MR90"/>
@@
 <attribute name="VALUE" x="33.525" y="24.15875" size="0.8128" layer="28" rot="MR180"/>
 </element>
-<element name="C8" library="my_rcl" package="C075" value="0.47u" x="38.1" y="32.385" smashed="yes">
+<element name="C8" library="my_rcl" package="C075" value="0.1u" x="38.1" y="32.385" smashed="yes">
 <attribute name="NAME" x="34.544" y="34.29" size="0.8128" layer="25" ratio="10"/>
 <attribute name="VALUE" x="38.354" y="29.49575" size="0.8128" layer="27" ratio="10"/>
@@
 <attribute name="VALUE" x="27.0925" y="13.64" size="0.8128" layer="28" rot="MR90"/>
 </element>
-<element name="C6" library="my_rcl" package="1608" value="1u" x="28.8925" y="11.1125" smashed="yes" rot="MR270">
+<element name="C6" library="my_rcl" package="1608" value="0.1u" x="28.8925" y="11.1125" smashed="yes" rot="MR270">
 <attribute name="NAME" x="27.8925" y="12.7125" size="0.8128" layer="26" rot="MR270"/>
 <attribute name="VALUE" x="27.0925" y="10.94125" size="0.8128" layer="28" rot="MR90"/>
@@
 <attribute name="VALUE" x="72.97125" y="7.6075" size="0.8128" layer="28" rot="MR90"/>
 </element>
-<element name="R23" library="my_rcl" package="1608" value="10k" x="69.85" y="4.7625" smashed="yes" rot="MR270">
+<element name="R23" library="my_rcl" package="1608" value="47k" x="69.85" y="4.7625" smashed="yes" rot="MR270">
 <attribute name="NAME" x="68.85" y="6.3625" size="0.8128" layer="26" rot="MR270"/>
 <attribute name="VALUE" x="71.80875" y="4.4575" size="0.8128" layer="28" rot="MR270"/>
 </element>
-<element name="R21" library="my_rcl" package="1608" value="10k" x="63.02375" y="5.715" smashed="yes" rot="MR270">
+<element name="R21" library="my_rcl" package="1608" value="1.5k" x="63.02375" y="5.715" smashed="yes" rot="MR270">
 <attribute name="NAME" x="62.02375" y="7.315" size="0.8128" layer="26" rot="MR270"/>
 <attribute name="VALUE" x="62.05875" y="3.705" size="0.8128" layer="28" rot="MR180"/>
@@
 <attribute name="VALUE" x="58.24875" y="9.42" size="0.8128" layer="28" rot="MR180"/>
 </element>
-<element name="R2" library="my_rcl" package="1608" value="120k" x="34.6075" y="5.3975" smashed="yes" rot="MR270">
+<element name="R2" library="my_rcl" package="1608" value="47k" x="34.6075" y="5.3975" smashed="yes" rot="MR270">
 <attribute name="NAME" x="33.6075" y="6.9975" size="0.8128" layer="26" rot="MR270"/>
 <attribute name="VALUE" x="34.97875" y="3.505" size="0.8128" layer="28" rot="MR270"/>
@@
 <attribute name="VALUE" x="31.01" y="3.505" size="0.8128" layer="28" rot="MR270"/>
 </element>
-<element name="R7" library="my_rcl" package="1608" value="250k" x="28.8925" y="5.3975" smashed="yes" rot="MR270">
+<element name="R7" library="my_rcl" package="1608" value="240k" x="28.8925" y="5.3975" smashed="yes" rot="MR270">
 <attribute name="NAME" x="27.8925" y="6.9975" size="0.8128" layer="26" rot="MR270"/>
 <attribute name="VALUE" x="29.26375" y="3.505" size="0.8128" layer="28" rot="MR270"/>
