File: acf-adapter.sch (EAGLE design)
At the start: 87 parts, among them IC1 UCC27712, IC2 UCC28780, IC3 TL431, Q1 TK8Q60, Q2 TK8Q60, Q3 2N7002, Q5 TLP621-1, T1 COMMON_FILTER-SU10VFC, T2 TRANSFORMAER_FLYBACK-PQ2620-A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

Commit message: できた
Parts:
- Q1: value TK8Q60 -> 2SK3115
- Q2: value TK8Q60 -> TK13A60
- Q4: value (none) -> BSS127
Changed lines of the file:
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@@
 <part name="IC1" library="my_ic" deviceset="UCC27712" device=""/>
 <part name="IC2" library="my_ic" deviceset="UCC28780" device=""/>
-<part name="Q1" library="my_ic" deviceset="NMOS" device="" value="TK8Q60"/>
-<part name="Q2" library="my_ic" deviceset="NMOS" device="" value="TK8Q60"/>
+<part name="Q1" library="my_ic" deviceset="NMOS" device="" value="2SK3115"/>
+<part name="Q2" library="my_ic" deviceset="NMOS" device="" value="TK13A60"/>
 <part name="R11" library="my_rcl" deviceset="R" device="-1608" value="10k"/>
 <part name="R12" library="my_rcl" deviceset="R" device="-1608" value="10k"/>
@@
 <part name="R5" library="my_rcl" deviceset="R" device="-1608" value="10k"/>
 <part name="R6" library="my_rcl" deviceset="R" device="-1608" value="47k"/>
-<part name="Q4" library="my_ic" deviceset="NMOS" device="-SMD"/>
+<part name="Q4" library="my_ic" deviceset="NMOS" device="-SMD" value="BSS127"/>
 <part name="C12" library="my_rcl" deviceset="C" device="-1608" value="100p"/>
 <part name="R7" library="my_rcl" deviceset="R" device="-1608" value="250k"/>

Commit message: 微修正
Parts:
- R16: value 100 -> 120
- R2: value 250k -> 125k
Changed lines of the file:
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@@
 <grid distance="0.05" unitdist="inch" unit="inch" style="lines" multiple="2" display="yes" altdistance="0.01" altunitdist="inch" altunit="inch"/>
 <layers>
-<layer number="1" name="Top" color="4" fill="1" visible="yes" active="no"/>
-<layer number="2" name="Route2" color="16" fill="1" visible="yes" active="no"/>
-<layer number="3" name="Route3" color="17" fill="1" visible="yes" active="no"/>
-<layer number="4" name="Route4" color="18" fill="1" visible="yes" active="no"/>
-<layer number="5" name="Route5" color="19" fill="1" visible="yes" active="no"/>
-<layer number="6" name="Route6" color="25" fill="1" visible="yes" active="no"/>
-<layer number="7" name="Route7" color="26" fill="1" visible="yes" active="no"/>
-<layer number="8" name="Route8" color="27" fill="1" visible="yes" active="no"/>
-<layer number="9" name="Route9" color="28" fill="1" visible="yes" active="no"/>
-<layer number="10" name="Route10" color="29" fill="1" visible="yes" active="no"/>
-<layer number="11" name="Route11" color="30" fill="1" visible="yes" active="no"/>
-<layer number="12" name="Route12" color="20" fill="1" visible="yes" active="no"/>
-<layer number="13" name="Route13" color="21" fill="1" visible="yes" active="no"/>
-<layer number="14" name="Route14" color="22" fill="1" visible="yes" active="no"/>
-<layer number="15" name="Route15" color="23" fill="1" visible="yes" active="no"/>
-<layer number="16" name="Bottom" color="1" fill="1" visible="yes" active="no"/>
-<layer number="17" name="Pads" color="2" fill="1" visible="yes" active="no"/>
-<layer number="18" name="Vias" color="2" fill="1" visible="yes" active="no"/>
-<layer number="19" name="Unrouted" color="6" fill="1" visible="yes" active="no"/>
-<layer number="20" name="Dimension" color="24" fill="1" visible="yes" active="no"/>
-<layer number="21" name="tPlace" color="7" fill="1" visible="yes" active="no"/>
-<layer number="22" name="bPlace" color="7" fill="1" visible="yes" active="no"/>
-<layer number="23" name="tOrigins" color="15" fill="1" visible="yes" active="no"/>
-<layer number="24" name="bOrigins" color="15" fill="1" visible="yes" active="no"/>
-<layer number="25" name="tNames" color="7" fill="1" visible="yes" active="no"/>
-<layer number="26" name="bNames" color="7" fill="1" visible="yes" active="no"/>
-<layer number="27" name="tValues" color="7" fill="1" visible="yes" active="no"/>
-<layer number="28" name="bValues" color="7" fill="1" visible="yes" active="no"/>
+<layer number="1" name="Top" color="4" fill="1" visible="no" active="no"/>
+<layer number="2" name="Route2" color="16" fill="1" visible="no" active="no"/>
+<layer number="3" name="Route3" color="17" fill="1" visible="no" active="no"/>
+<layer number="4" name="Route4" color="18" fill="1" visible="no" active="no"/>
+<layer number="5" name="Route5" color="19" fill="1" visible="no" active="no"/>
+<layer number="6" name="Route6" color="25" fill="1" visible="no" active="no"/>
+<layer number="7" name="Route7" color="26" fill="1" visible="no" active="no"/>
+<layer number="8" name="Route8" color="27" fill="1" visible="no" active="no"/>
+<layer number="9" name="Route9" color="28" fill="1" visible="no" active="no"/>
+<layer number="10" name="Route10" color="29" fill="1" visible="no" active="no"/>
+<layer number="11" name="Route11" color="30" fill="1" visible="no" active="no"/>
+<layer number="12" name="Route12" color="20" fill="1" visible="no" active="no"/>
+<layer number="13" name="Route13" color="21" fill="1" visible="no" active="no"/>
+<layer number="14" name="Route14" color="22" fill="1" visible="no" active="no"/>
+<layer number="15" name="Route15" color="23" fill="1" visible="no" active="no"/>
+<layer number="16" name="Bottom" color="1" fill="1" visible="no" active="no"/>
+<layer number="17" name="Pads" color="2" fill="1" visible="no" active="no"/>
+<layer number="18" name="Vias" color="2" fill="1" visible="no" active="no"/>
+<layer number="19" name="Unrouted" color="6" fill="1" visible="no" active="no"/>
+<layer number="20" name="Dimension" color="24" fill="1" visible="no" active="no"/>
+<layer number="21" name="tPlace" color="7" fill="1" visible="no" active="no"/>
+<layer number="22" name="bPlace" color="7" fill="1" visible="no" active="no"/>
+<layer number="23" name="tOrigins" color="15" fill="1" visible="no" active="no"/>
+<layer number="24" name="bOrigins" color="15" fill="1" visible="no" active="no"/>
+<layer number="25" name="tNames" color="7" fill="1" visible="no" active="no"/>
+<layer number="26" name="bNames" color="7" fill="1" visible="no" active="no"/>
+<layer number="27" name="tValues" color="7" fill="1" visible="no" active="no"/>
+<layer number="28" name="bValues" color="7" fill="1" visible="no" active="no"/>
 <layer number="29" name="tStop" color="7" fill="3" visible="no" active="no"/>
 <layer number="30" name="bStop" color="7" fill="6" visible="no" active="no"/>
@@
 <layer number="35" name="tGlue" color="7" fill="4" visible="no" active="no"/>
 <layer number="36" name="bGlue" color="7" fill="5" visible="no" active="no"/>
-<layer number="37" name="tTest" color="7" fill="1" visible="yes" active="no"/>
-<layer number="38" name="bTest" color="7" fill="1" visible="yes" active="no"/>
+<layer number="37" name="tTest" color="7" fill="1" visible="no" active="no"/>
+<layer number="38" name="bTest" color="7" fill="1" visible="no" active="no"/>
 <layer number="39" name="tKeepout" color="4" fill="11" visible="no" active="no"/>
 <layer number="40" name="bKeepout" color="1" fill="11" visible="no" active="no"/>
@@
 <layer number="44" name="Drills" color="7" fill="1" visible="no" active="no"/>
 <layer number="45" name="Holes" color="7" fill="1" visible="no" active="no"/>
-<layer number="46" name="Milling" color="3" fill="1" visible="yes" active="no"/>
-<layer number="47" name="Measures" color="7" fill="1" visible="yes" active="no"/>
-<layer number="48" name="Document" color="7" fill="1" visible="yes" active="no"/>
-<layer number="49" name="Reference" color="7" fill="1" visible="yes" active="no"/>
-<layer number="50" name="dxf" color="7" fill="1" visible="yes" active="no"/>
-<layer number="51" name="tDocu" color="7" fill="1" visible="yes" active="no"/>
-<layer number="52" name="bDocu" color="7" fill="1" visible="yes" active="no"/>
-<layer number="53" name="tGND_GNDA" color="7" fill="1" visible="yes" active="no"/>
-<layer number="54" name="bGND_GNDA" color="7" fill="1" visible="yes" active="no"/>
-<layer number="56" name="wert" color="7" fill="1" visible="yes" active="no"/>
-<layer number="57" name="tCAD" color="7" fill="1" visible="yes" active="no"/>
-<layer number="59" name="tCarbon" color="7" fill="1" visible="yes" active="no"/>
-<layer number="60" name="bCarbon" color="7" fill="1" visible="yes" active="no"/>
+<layer number="46" name="Milling" color="3" fill="1" visible="no" active="no"/>
+<layer number="47" name="Measures" color="7" fill="1" visible="no" active="no"/>
+<layer number="48" name="Document" color="7" fill="1" visible="no" active="no"/>
+<layer number="49" name="Reference" color="7" fill="1" visible="no" active="no"/>
+<layer number="50" name="dxf" color="7" fill="1" visible="no" active="no"/>
+<layer number="51" name="tDocu" color="7" fill="1" visible="no" active="no"/>
+<layer number="52" name="bDocu" color="7" fill="1" visible="no" active="no"/>
+<layer number="53" name="tGND_GNDA" color="7" fill="1" visible="no" active="no"/>
+<layer number="54" name="bGND_GNDA" color="7" fill="1" visible="no" active="no"/>
+<layer number="56" name="wert" color="7" fill="1" visible="no" active="no"/>
+<layer number="57" name="tCAD" color="7" fill="1" visible="no" active="no"/>
+<layer number="59" name="tCarbon" color="7" fill="1" visible="no" active="no"/>
+<layer number="60" name="bCarbon" color="7" fill="1" visible="no" active="no"/>
 <layer number="88" name="SimResults" color="9" fill="1" visible="yes" active="yes"/>
 <layer number="89" name="SimProbes" color="9" fill="1" visible="yes" active="yes"/>
@@
 <part name="C8" library="my_rcl" deviceset="C" device="-7.5" value="0.47u"/>
 <part name="R1" library="my_rcl" deviceset="R" device="-1608" value="250k"/>
-<part name="R2" library="my_rcl" deviceset="R" device="-1608" value="250k"/>
+<part name="R2" library="my_rcl" deviceset="R" device="-1608" value="125k"/>
 <part name="R4" library="my_rcl" deviceset="R" device="-1608" value="47k"/>
 <part name="C3" library="my_rcl" deviceset="C" device="-1608" value="0.1u"/>
@@
 <part name="C11" library="my_rcl" deviceset="C" device="-2012" value="10u"/>
 <part name="R18" library="my_rcl" deviceset="R" device="-1608" value="10"/>
-<part name="R16" library="my_rcl" deviceset="R" device="-1608" value="100"/>
+<part name="R16" library="my_rcl" deviceset="R" device="-1608" value="120"/>
 <part name="C10" library="my_rcl" deviceset="C" device="-1608" value="27p"/>
 <part name="R14" library="my_rcl" deviceset="R" device="-1608" value="1M"/>

Commit message: 発注
Parts:
- added R30: 240k, my_rcl:R-1608
- R1: value 250k -> 240k
- R14: value 1M -> 240k
- R15: value 470k -> 240k
- R2: value 125k -> 120k
- R27: value 10 -> 120
- R8, R9: device my_rcl:R-1608 -> my_rcl:R-2012
Connections:
- new net N$37: R15.1, R30.1
- net N$34: now also R30.2; no longer R15.1

Commit message: 微修正
Parts:
- C11: value 10u -> 47u
- C6: value 1u -> 0.1u
- C8: value 0.47u -> 0.1u
- R2: value 120k -> 47k
- R21: value 10k -> 1.5k
- R23: value 10k -> 47k
- R7: value 250k -> 240k
